File: _autosave-_autosave-microboard.kicad_pcb (KiCad board)
At the start: 2 copper layers, 121.9 x 68.6 mm, 95 parts, among them J10 Conn_01x01, J11 Conn_01x01, J12 Conn_01x10, J13 Conn_01x01, J14 Conn_01x12, J15 Conn_01x03, J17 Conn_01x01, J18 Conn_01x01, J2 Conn_01x10, J21 Conn_01x01_Socket, J22 Conn_01x01_Socket, J3 Conn_02x12, J39 Conn_01x10, J4 USB4085-GF-A_REVB, J40 Conn_01x10, J41 Conn_01x10, J43 Conn_01x05, J44 Conn_01x09, J45 Conn_01x08, J5 Conn_01x04, J6 Conn_01x04, J7 Conn_01x05, J8 Conn_01x10, J9 Conn_01x01, SW1 SW_Push, SW2 SW_Push, SW7 RotaryEncoder_Switch, U1 USBLC6-2SC6, U2 ATSAMD21G18A-AUT, U3 LF33_TO220, U7 LF50_TO220, Y1 32768Hz

Commit message: small msg
Parts:
- moved J44 1.33 mm to (190.2, 96.5)
- moved J45 1.33 mm to (206.0, 96.4)
Routing:
- net Net-(J8-Pin_2): track 0.00 -> 7.82 mm
- net Net-(J8-Pin_1): track 0.00 -> 7.82 mm
- net GND: track 647.7 -> 655.0 mm
- net Net-(BAR1-A-Pad9): track 0.00 -> 3.12 mm
- net Net-(BAR1-A-Pad10): track 0.00 -> 3.12 mm
- net +5V: track 207.1 -> 207.8 mm
- net +3.3V: track 429.6 -> 430.2 mm
