File: microboard.kicad_pcb (KiCad board)
At the start: 2 copper layers, 95 parts, among them J1 Conn_01x01, J10 Conn_01x01, J11 Conn_01x01, J12 Conn_01x10, J13 Conn_01x01, J17 Conn_01x01, J18 Conn_01x01, J2 Conn_01x10, J21 Conn_01x01_Socket, J22 Conn_01x01_Socket, J24 Conn_01x01, J25 Conn_01x01, J3 Conn_02x12, J39 Conn_01x10, J4 USB_C_Receptacle_USB2.0, J40 Conn_01x10, J41 Conn_01x10, J43 Conn_01x05, J44 Conn_01x09, J45 Conn_01x08, J5 Conn_01x04, J6 Conn_01x04, J7 Conn_01x05, J8 Conn_01x10, J9 Conn_01x01, SW1 SW_Push, SW3 SW_Push, SW4 SW_Push, SW7 RotaryEncoder_Switch, U1 USBLC6-2SC6, U2 ATSAMD21G18A-AUT, U3 LF33_TO220, U4 TXS0108EPW, U7 LF50_TO220, Y1 32768Hz

Commit message: update
Parts:
- removed C19, C21, C22: 0.1uF, Capacitor_SMD:C_0805_2012Metric_Pad1.18x1.45mm_HandSolder
- removed R10, R11, R5: 22K, Resistor_SMD:R_0805_2012Metric_Pad1.20x1.40mm_HandSolder
- moved H4 19.3 mm to (242.7, 120.5)
- moved H1 18.1 mm to (242.6, 59.4)
- moved H2 16.7 mm to (130.6, 59.2)
- moved H3 16.2 mm to (130.7, 120.6)
- moved BAR1 3.81 mm to (229.9, 59.7)
- moved D4 2.81 mm to (136.2, 60.8)
- moved R3 2.81 mm to (136.2, 58.3)
- moved R14 2.54 mm to (224.7, 59.7)
- moved R15 2.54 mm to (224.7, 62.2)
- moved R16 2.54 mm to (224.7, 64.8)
- moved R17 2.54 mm to (224.7, 67.3)
- moved R19 2.54 mm to (224.7, 72.4)
- moved R20 2.54 mm to (224.7, 74.9)
- moved R21 2.54 mm to (224.7, 77.5)
- moved R22 2.54 mm to (224.7, 80.0)
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- renumbered SW1 to RESET1, SW3 to SW1, SW4 to SW2
Connections:
- J12 pad 10: GND -> Net-(J12-Pin_10)
- J12 pad 11: +3.3V -> Net-(J12-Pin_11)
- J12 pad 12: Net-(J12-Pin_12) -> Net-(J12-Pin_11)
- J12 pad 14: Net-(J12-Pin_14) -> Net-(J12-Pin_13)
- J12 pad 16: Net-(J12-Pin_16) -> Net-(J12-Pin_15)
- J12 pad 18: Net-(J12-Pin_18) -> Net-(J12-Pin_17)
- J12 pad 19: Net-(J12-Pin_19) -> GND
- J12 pad 2: Net-(J12-Pin_12) -> +3.3V
- J12 pad 3: Net-(J12-Pin_13) -> Net-(J12-Pin_3)
- J12 pad 4: Net-(J12-Pin_14) -> Net-(J12-Pin_3)
- J12 pad 5: Net-(J12-Pin_15) -> Net-(J12-Pin_5)
- J12 pad 6: Net-(J12-Pin_16) -> Net-(J12-Pin_5)
- J12 pad 7: Net-(J12-Pin_17) -> Net-(J12-Pin_7)
- J12 pad 8: Net-(J12-Pin_18) -> Net-(J12-Pin_7)
- J12 pad 9: Net-(J12-Pin_19) -> Net-(J12-Pin_10)
- J2 pad 10: GND -> Net-(J2-Pin_10)
- J2 pad 11: +3.3V -> Net-(J2-Pin_11)
- J2 pad 12: Net-(J2-Pin_12) -> Net-(J2-Pin_11)
- J2 pad 14: Net-(J2-Pin_14) -> Net-(J2-Pin_13)
- J2 pad 16: Net-(J2-Pin_16) -> Net-(J2-Pin_15)
- J2 pad 18: Net-(J2-Pin_18) -> Net-(J2-Pin_17)
- J2 pad 19: Net-(J2-Pin_19) -> GND
- J2 pad 2: Net-(J2-Pin_12) -> +3.3V
- J2 pad 3: Net-(J2-Pin_13) -> Net-(J2-Pin_3)
- J2 pad 4: Net-(J2-Pin_14) -> Net-(J2-Pin_3)
- J2 pad 5: Net-(J2-Pin_15) -> Net-(J2-Pin_5)
- J2 pad 6: Net-(J2-Pin_16) -> Net-(J2-Pin_5)
- J2 pad 7: Net-(J2-Pin_17) -> Net-(J2-Pin_7)
- J2 pad 8: Net-(J2-Pin_18) -> Net-(J2-Pin_7)
- J2 pad 9: Net-(J2-Pin_19) -> Net-(J2-Pin_10)
- J39 pad 1: Net-(D8-K) -> +3.3V
- J39 pad 10: Net-(D8-K) -> +3.3V
- J39 pad 2: Net-(D8-K) -> +3.3V
- J39 pad 3: Net-(D8-K) -> +3.3V
- J39 pad 4: Net-(D8-K) -> +3.3V
- J39 pad 5: Net-(D8-K) -> +3.3V
- J39 pad 6: Net-(D8-K) -> +3.3V
- J39 pad 7: Net-(D8-K) -> +3.3V
- J39 pad 8: Net-(D8-K) -> +3.3V
- J39 pad 9: Net-(D8-K) -> +3.3V
- J40 pad 1: Net-(D9-K) -> +5V
- J40 pad 10: Net-(D9-K) -> +5V
- J40 pad 2: Net-(D9-K) -> +5V
- J40 pad 3: Net-(D9-K) -> +5V
- J40 pad 4: Net-(D9-K) -> +5V
- J40 pad 5: Net-(D9-K) -> +5V
- J40 pad 6: Net-(D9-K) -> +5V
- J40 pad 7: Net-(D9-K) -> +5V
- J40 pad 8: Net-(D9-K) -> +5V
- J40 pad 9: Net-(D9-K) -> +5V
- J43 pad 10: GND -> Net-(J43-Pin_10)
- J43 pad 11: +3.3V -> Net-(J43-Pin_11)
- J43 pad 12: Net-(J43-Pin_12) -> Net-(J43-Pin_11)
- J43 pad 14: Net-(J43-Pin_14) -> Net-(J43-Pin_13)
- J43 pad 16: Net-(J43-Pin_16) -> Net-(J43-Pin_15)
- J43 pad 17: Net-(J43-Pin_17) -> GND
- J43 pad 18: Net-(J43-Pin_18) -> GND
- J43 pad 2: Net-(J43-Pin_12) -> +3.3V
- J43 pad 3: Net-(J43-Pin_13) -> Net-(J43-Pin_3)
- J43 pad 4: Net-(J43-Pin_14) -> Net-(J43-Pin_3)
- J43 pad 5: Net-(J43-Pin_15) -> Net-(J43-Pin_5)
- J43 pad 6: Net-(J43-Pin_16) -> Net-(J43-Pin_5)
- J43 pad 7: Net-(J43-Pin_17) -> Net-(J43-Pin_7)
- J43 pad 8: Net-(J43-Pin_18) -> Net-(J43-Pin_7)
- J43 pad 9: GND -> Net-(J43-Pin_10)
- J7 pad 1: Net-(J43-Pin_18) -> Net-(J43-Pin_15)
- J7 pad 2: Net-(J43-Pin_17) -> Net-(J43-Pin_13)
- SW7 pad A: Net-(R5-Pad2) -> Net-(J6-Pin_3)
- SW7 pad B: Net-(R11-Pad2) -> Net-(J6-Pin_2)
- SW7 pad S1: Net-(R10-Pad2) -> Net-(J6-Pin_4)
- U2 pad 14: Net-(J12-Pin_12) -> Net-(J12-Pin_3)
- U2 pad 15: Net-(J12-Pin_13) -> Net-(J12-Pin_5)
- U2 pad 16: Net-(J12-Pin_14) -> Net-(J12-Pin_7)
- U2 pad 19: Net-(J12-Pin_15) -> Net-(J12-Pin_10)
- U2 pad 20: Net-(J12-Pin_16) -> Net-(J12-Pin_11)
- U2 pad 21: Net-(J12-Pin_17) -> Net-(J12-Pin_13)
- U2 pad 22: Net-(J12-Pin_18) -> Net-(J12-Pin_15)
- U2 pad 23: Net-(J12-Pin_19) -> Net-(J12-Pin_17)
- U2 pad 24: Net-(J2-Pin_12) -> Net-(J2-Pin_3)
- U2 pad 25: Net-(J2-Pin_13) -> Net-(J2-Pin_5)
- U2 pad 26: Net-(J2-Pin_14) -> Net-(J2-Pin_7)
- U2 pad 27: Net-(J2-Pin_15) -> Net-(J2-Pin_10)
- U2 pad 28: Net-(J2-Pin_16) -> Net-(J2-Pin_11)
- U2 pad 29: Net-(J2-Pin_17) -> Net-(J2-Pin_13)
- U2 pad 30: Net-(J2-Pin_18) -> Net-(J2-Pin_15)
- U2 pad 31: Net-(J2-Pin_19) -> Net-(J2-Pin_17)
- U2 pad 32: Net-(J43-Pin_12) -> Net-(J43-Pin_3)
- U2 pad 37: Net-(J43-Pin_13) -> Net-(J43-Pin_5)
- U2 pad 38: Net-(J43-Pin_14) -> Net-(J43-Pin_7)
- U2 pad 39: Net-(J43-Pin_15) -> Net-(J43-Pin_10)
- U2 pad 41: Net-(J43-Pin_16) -> Net-(J43-Pin_11)
- U2 pad 45: Net-(J43-Pin_17) -> Net-(J43-Pin_13)
- U2 pad 46: Net-(J43-Pin_18) -> Net-(J43-Pin_15)

Commit message: paths
Parts:
- removed D9: D, Diode_SMD:D_SOD-323_HandSoldering
- removed J1, J24, J25: Conn_01x01, Connector_PinHeader_2.54mm:PinHeader_1x01_P2.54mm_Vertical
- removed U4: TXS0108EPW, Package_SO:TSSOP-20_4.4x6.5mm_P0.65mm
- added C19: 22nF, Capacitor_SMD:C_0805_2012Metric_Pad1.18x1.45mm_HandSolder, F.Cu at (194.3, 108.2)
- added D5: LED, LED_SMD:LED_0805_2012Metric_Pad1.15x1.40mm_HandSolder, F.Cu at (177.8, 76.2)
- added D8: LED, LED_SMD:LED_0805_2012Metric_Pad1.15x1.40mm_HandSolder, F.Cu at (181.6, 76.2)
- added J14: Conn_01x12, Connector_PinHeader_2.54mm:PinHeader_1x12_P2.54mm_Vertical, F.Cu at (228.6, 119.4)
- added J15: Conn_01x03, Connector_PinHeader_2.54mm:PinHeader_1x03_P2.54mm_Vertical, F.Cu at (190.5, 119.4)
- added JP1: SolderJumper_2_Open, Jumper:SolderJumper-2_P1.3mm_Open_RoundedPad1.0x1.5mm, F.Cu at (193.0, 113.0)
- added R10: 1k, Resistor_SMD:R_0805_2012Metric_Pad1.20x1.40mm_HandSolder, F.Cu at (178.1, 81.3)
- added R11: 1k, Resistor_SMD:R_0805_2012Metric_Pad1.20x1.40mm_HandSolder, F.Cu at (181.6, 81.3)
- added R4: 10, Resistor_SMD:R_0805_2012Metric_Pad1.20x1.40mm_HandSolder, F.Cu at (193.0, 104.4)
- added R5: 10, Resistor_SMD:R_0805_2012Metric_Pad1.20x1.40mm_HandSolder, F.Cu at (191.8, 108.2)
- added RV1: R_Potentiometer_Trim, Potentiometer_THT:Potentiometer_Runtron_RM-065_Vertical, F.Cu at (205.7, 114.0)
- J44: footprint Connector_PinHeader_2.54mm:PinHeader_1x09_P2.54mm_Vertical -> Connector_PinHeader_2.54mm:PinHeader_1x10_P2.54mm_Vertical
- J45: footprint Connector_PinHeader_2.54mm:PinHeader_1x08_P2.54mm_Vertical -> Connector_PinHeader_2.54mm:PinHeader_2x10_P2.54mm_Vertical
- moved J21 53.1 mm to (245.1, 68.6), turned to 180 degrees
- moved J22 46.0 mm to (245.1, 80.0), turned to 180 degrees
- moved J10 33.3 mm to (244.1, 111.8), turned to 90 degrees
- moved J44 29.5 mm to (218.4, 86.4), turned to 90 degrees
- moved J11 28.2 mm to (223.5, 111.8), turned to 90 degrees
- moved C4 26.8 mm to (146.1, 87.9), turned to -90 degrees
- moved SW2 25.5 mm to (237.5, 111.8), turned to 90 degrees
- moved J45 22.4 mm to (218.3, 104.6), turned to 90 degrees
- moved SW1 20.5 mm to (217.2, 111.8), turned to 90 degrees
- moved J18 19.4 mm to (231.1, 111.8), turned to 90 degrees
- moved R6 19.2 mm to (149.9, 87.9), turned to 90 degrees
- moved J17 14.5 mm to (210.8, 111.8), turned to 90 degrees
- moved H1 2.56 mm to (245.1, 59.7)
- moved H4 2.43 mm to (245.1, 120.5)
- moved C2 1.27 mm to (144.0, 100.9), turned to 0 degrees
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Connections:
- J43 pad 17: GND -> Net-(J43-Pin_17)
- J43 pad 18: GND -> Net-(J43-Pin_17)
- J44 pad 1: Net-(J44-Pin_1) -> +3.3V
- J44 pad 2: Net-(J44-Pin_2) -> +3.3V
- J44 pad 3: Net-(J44-Pin_3) -> +3.3V
- J44 pad 4: Net-(J44-Pin_4) -> +3.3V
- J44 pad 5: Net-(J44-Pin_5) -> +3.3V
- J44 pad 6: Net-(J44-Pin_6) -> +3.3V
- J44 pad 7: Net-(J44-Pin_7) -> +3.3V
- J44 pad 8: Net-(J44-Pin_8) -> +3.3V
- J44 pad 9: Net-(J44-Pin_9) -> +3.3V
- J45 pad 2: Net-(J45-Pin_2) -> Net-(J45-Pin_1)
- J45 pad 4: Net-(J45-Pin_4) -> Net-(J45-Pin_3)
- J45 pad 6: Net-(J45-Pin_6) -> Net-(J45-Pin_5)
- J45 pad 8: Net-(J45-Pin_8) -> Net-(J45-Pin_7)
- J7 pad 1: Net-(J43-Pin_15) -> Net-(J43-Pin_17)
- J7 pad 2: Net-(J43-Pin_13) -> Net-(J43-Pin_15)
- U2 pad 13: +3.3V -> Net-(J12-Pin_3)
- U2 pad 14: Net-(J12-Pin_3) -> Net-(J12-Pin_5)
- U2 pad 15: Net-(J12-Pin_5) -> Net-(J12-Pin_7)
- U2 pad 16: Net-(J12-Pin_7) -> Net-(J12-Pin_10)
- U2 pad 19: Net-(J12-Pin_10) -> Net-(J12-Pin_11)
- U2 pad 20: Net-(J12-Pin_11) -> Net-(J12-Pin_13)
- U2 pad 21: Net-(J12-Pin_13) -> Net-(J12-Pin_15)
- U2 pad 22: Net-(J12-Pin_15) -> Net-(J12-Pin_17)
- U2 pad 23: Net-(J12-Pin_17) -> Net-(J2-Pin_3)
- U2 pad 24: Net-(J2-Pin_3) -> Net-(J2-Pin_5)
- U2 pad 25: Net-(J2-Pin_5) -> Net-(J2-Pin_7)
- U2 pad 26: Net-(J2-Pin_7) -> Net-(J2-Pin_10)
- U2 pad 27: Net-(J2-Pin_10) -> Net-(J2-Pin_11)
- U2 pad 28: Net-(J2-Pin_11) -> Net-(J2-Pin_13)
- U2 pad 29: Net-(J2-Pin_13) -> Net-(J2-Pin_15)
- U2 pad 30: Net-(J2-Pin_15) -> Net-(J2-Pin_17)
- U2 pad 31: Net-(J2-Pin_17) -> Net-(J43-Pin_3)
- U2 pad 32: Net-(J43-Pin_3) -> Net-(J43-Pin_5)
- U2 pad 37: Net-(J43-Pin_5) -> Net-(J43-Pin_7)
- U2 pad 38: Net-(J43-Pin_7) -> Net-(J43-Pin_10)
- U2 pad 39: Net-(J43-Pin_10) -> Net-(J43-Pin_11)
- U2 pad 41: Net-(J43-Pin_11) -> Net-(J43-Pin_13)
- U2 pad 45: Net-(J43-Pin_13) -> Net-(J43-Pin_15)
- U2 pad 46: Net-(J43-Pin_15) -> Net-(J43-Pin_17)
Routing:
- net GND: track 0.00 -> 613.9 mm, vias 0 -> 2
- net +3.3V: track 0.00 -> 315.9 mm, vias 0 -> 4
- net +5V: track 0.00 -> 139.5 mm
- net USBrail: track 0.00 -> 71.4 mm, vias 0 -> 1
- net RESET: track 0.00 -> 63.0 mm, vias 0 -> 2
- net Net-(J3-Pin_5): track 0.00 -> 50.4 mm, vias 0 -> 3
- net Net-(J3-Pin_3): track 0.00 -> 44.1 mm, vias 0 -> 2
- net Net-(J3-Pin_21): track 0.00 -> 38.3 mm
- net Net-(J6-Pin_4): track 0.00 -> 37.8 mm
- net AREF: track 0.00 -> 36.3 mm
- net Net-(J14-Pin_2): track 0.00 -> 35.9 mm
- net Net-(J12-Pin_15): track 0.00 -> 35.2 mm, vias 0 -> 1
- net Net-(J43-Pin_17): track 0.00 -> 33.8 mm
- net Net-(J43-Pin_15): track 0.00 -> 32.0 mm
- net Net-(J3-Pin_10): track 0.00 -> 30.9 mm, vias 0 -> 1
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- added copper zone on B.Cu, net GND
- added copper zone on F.Cu, net GND

Commit message: almost final design
Parts:
- J4: value USB_C_Receptacle_USB2.0 -> USB4085-GF-A_REVB; footprint Connector_USB:USB_C_Receptacle_GCT_USB4105-xx-A_16P_TopMnt_Horizontal -> usb4085:GCT_USB4085-GF-A_REVB
- moved J4 38.9 mm to (91.4, 77.0)
- moved H2 38.5 mm to (93.3, 68.4)
- moved H4 38.4 mm to (207.8, 129.4)
- moved J12 38.4 mm to (108.7, 128.3)
- moved J15 38.4 mm to (153.1, 128.3)
- moved R15 38.4 mm to (187.3, 71.1)
- moved BAR1 38.4 mm to (192.5, 68.6)
- moved C1 38.4 mm to (153.1, 80.0)
- moved C11 38.4 mm to (119.2, 119.9)
- moved C13 38.4 mm to (101.1, 86.4)
- moved C16 38.4 mm to (140.4, 78.7)
- moved C17 38.4 mm to (118.8, 77.5)
- moved C18 38.4 mm to (118.8, 80.0)
- moved C19 38.4 mm to (156.9, 117.1)
- moved C20 38.4 mm to (140.4, 81.3)
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- renumbered RESET1 to RESET
Connections:
- C13 pad 1: Net-(J4-SHIELD) -> Net-(C13-Pad1)
- J14 pad 6: Pa28 -> PA28
- J2 pad 11: Net-(J2-Pin_11) -> PA18
- J2 pad 12: Net-(J2-Pin_11) -> PA18
- J2 pad 13: Net-(J2-Pin_13) -> PA19
- J2 pad 14: Net-(J2-Pin_13) -> PA19
- J2 pad 15: Net-(J2-Pin_15) -> PA20
- J2 pad 16: Net-(J2-Pin_15) -> PA20
- J2 pad 17: Net-(J2-Pin_17) -> PA21
- J2 pad 18: Net-(J2-Pin_17) -> PA21
- J4 pad A6: Net-(J5-Pin_2) -> D-
- J4 pad A7: Net-(J5-Pin_3) -> D+
- J4 pad B6: Net-(J5-Pin_2) -> D-
- J4 pad B7: Net-(J5-Pin_3) -> D+
- J4 pad S1: Net-(J4-SHIELD) -> Net-(C13-Pad1)
- J43 pad 11: Net-(J43-Pin_11) -> PA27
- J43 pad 12: Net-(J43-Pin_11) -> PA27
- J43 pad 13: Net-(J43-Pin_13) -> PA28
- J43 pad 14: Net-(J43-Pin_13) -> PA28
- J43 pad 15: Net-(J43-Pin_15) -> PA30
- J43 pad 16: Net-(J43-Pin_15) -> PA30
- J43 pad 17: Net-(J43-Pin_17) -> PA31
- J43 pad 18: Net-(J43-Pin_17) -> PA31
- J7 pad 1: Net-(J43-Pin_17) -> PA31
- J7 pad 2: Net-(J43-Pin_15) -> PA30
- R12 pad 1: Net-(J4-SHIELD) -> Net-(C13-Pad1)
- U2 pad 27: Net-(J2-Pin_11) -> PA18
- U2 pad 28: Net-(J2-Pin_13) -> PA19
- U2 pad 29: Net-(J2-Pin_15) -> PA20
- U2 pad 30: Net-(J2-Pin_17) -> PA21
- U2 pad 39: Net-(J43-Pin_11) -> PA27
- U2 pad 41: Net-(J43-Pin_13) -> PA28
- U2 pad 45: Net-(J43-Pin_15) -> PA30
- U2 pad 46: Net-(J43-Pin_17) -> PA31
Routing:
- net PA27: track 0.00 -> 179.1 mm
- net PA28: track 0.00 -> 129.6 mm, vias 0 -> 2
- net PA31: track 0.00 -> 91.8 mm, vias 0 -> 4
- net D+: track 0.00 -> 89.6 mm, vias 0 -> 4
- net D-: track 0.00 -> 86.4 mm, vias 0 -> 4
- net PA30: track 0.00 -> 77.6 mm, vias 0 -> 4
- net PA21: track 0.00 -> 74.6 mm, vias 0 -> 2
- net PA20: track 0.00 -> 70.2 mm, vias 0 -> 1
- net PA18: track 0.00 -> 67.4 mm, vias 0 -> 1
- net PA19: track 0.00 -> 66.5 mm, vias 0 -> 1
- net GND: track 613.9 -> 673.0 mm, vias 2 -> 5
- net Net-(J43-Pin_17): track 33.8 -> 0.00 mm
- net Net-(J43-Pin_15): track 32.0 -> 0.00 mm
- net Net-(C13-Pad1): track 0.00 -> 31.6 mm, vias 0 -> 2
- net Net-(J2-Pin_17): track 25.5 -> 0.00 mm
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Other:
- board outline added: 121.9 x 68.6 mm
- board text added: "0"
- board text added: "1"
- board text added: "10"
- board text added: "11"
- board text added: "12"
- board text added: "13"
- board text added: "14"
- board text added: "15"
- board text added: "16"
- board text added: "17"
- board text added: "18"
- board text added: "19"
- board text added: "2"
- board text added: "20"
- board text added: "21"
- board text added: "22"
- board text added: "23"
- board text added: "24"
- board text added: "25"
- board text added: "26"
- board text added: "27"
- board text added: "3"
- board text added: "3.3 V"
- board text added: "3.3V"
- board text added: "4"
- board text added: "5"
- board text added: "5V"
- board text added: "6"
- board text added: "7"
- board text added: "8"
- board text added: "9"
- board text added: "A/C"
- board text added: "A0"
- board text added: "A2"
- board text added: "A3"
- board text added: "A4"
- board text added: "A5"
- board text added: "AREF"
- board text added: "CON"
- board text added: "D1"
- board text added: "D2"
- board text added: "D3"
- board text added: "D4"
- board text added: "ENA"
- board text added: "GND"
- board text added: "HV"
- board text added: "LED"
- board text added: "LEVEL CONVERTER"
- board text added: "LV"
- board text added: "R/W"
- board text added: "RS"
- board text added: "SCL"
- board text added: "SDA"
- board text added: "SWCLK"
- board text added: "SWDIO"
- board text added: "VDD"

Commit message: new update just dropped!
Parts:
- J44: footprint Connector_PinHeader_2.54mm:PinHeader_1x10_P2.54mm_Vertical -> Connector_PinHeader_2.54mm:PinHeader_2x10_P2.54mm_Vertical
- RESET1: renamed from RESET; footprint Button_Switch_SMD:SW_Push_1P1T_NO_6x6mm_H9.5mm -> Button_Switch_THT:SW_PUSH_6mm_H8mm
- SW1, SW2: footprint Button_Switch_SMD:SW_Push_1P1T_NO_6x6mm_H9.5mm -> Button_Switch_THT:SW_PUSH_6mm_H8mm
- moved BAR1 34.8 mm to (166.2, 91.3), turned to 180 degrees
- moved J45 31.1 mm to (206.0, 95.1), turned to 0 degrees
- moved R23 28.0 mm to (171.4, 68.4), turned to 180 degrees
- moved R14 27.7 mm to (171.4, 91.3), turned to 180 degrees
- moved SW2 27.7 mm to (179.9, 101.7), turned to 0 degrees
- moved J14 27.6 mm to (163.6, 128.1), turned to 90 degrees
- moved J18 25.9 mm to (183.2, 97.1), turned to 0 degrees
- moved J40 25.9 mm to (200.5, 68.3)
- moved J39 25.7 mm to (185.1, 68.4)
- moved J41 25.7 mm to (192.7, 68.4)
- moved J10 25.7 mm to (183.2, 110.5), turned to 0 degrees
- moved R22 24.0 mm to (171.4, 70.9), turned to 180 degrees
- moved R15 23.8 mm to (171.4, 88.7), turned to 180 degrees
- moved J8 23.1 mm to (177.7, 68.5), turned to 0 degrees
- moved R21 20.5 mm to (171.4, 73.5), turned to 180 degrees
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Routing:
- net +3.3V: track 335.3 -> 429.6 mm, vias 6 -> 8
- net +5V: track 139.5 -> 207.1 mm
- net Net-(J14-Pin_11): track 18.8 -> 40.6 mm, vias 0 -> 1
- net PA21: track 74.6 -> 92.1 mm, vias 2 -> 1
- net PA20: track 70.2 -> 83.2 mm
- net D+: track 89.6 -> 76.9 mm
- net PA27: track 179.1 -> 166.8 mm
- net PA19: track 66.5 -> 75.7 mm, vias 1 -> 2
- net Net-(J14-Pin_3): track 24.6 -> 18.0 mm, vias 0 -> 1
- net PA18: track 67.4 -> 71.0 mm, vias 1 -> 2
- net GND: track 673.0 -> 676.0 mm
- net PA28: track 129.6 -> 127.3 mm, vias 2 -> 3
- net RESET: track 63.0 -> 61.0 mm
- net Net-(J10-Pin_1): track 12.0 -> 10.3 mm
- net Net-(J14-Pin_2): track 35.9 -> 34.9 mm
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Other:
- board text added: "30"
- board text added: "31"
- board text added: "38"
- board text added: "42"
- board text added: "44"
- board text added: "45"
- board text added: "Ano"
- board text added: "PA02"
- board text added: "PA03"
- board text added: "PA04"
- board text added: "PA05"
- board text added: "PA06"
- board text added: "PA07"
- board text added: "PA08"
- board text added: "PA09"
- board text added: "PA10"
- board text added: "PA11"
- board text added: "PA12"
- board text added: "PA13"
- board text added: "PA14"
- board text added: "PA15"
- board text added: "PA16"
- board text added: "PA17"
- board text added: "PA18"
- board text added: "PA19"
- board text added: "PA20"
- board text added: "PA21"
- board text added: "PA22"
- board text added: "PA23"
- board text added: "PA27"
- board text added: "PA28"
- board text added: "PA30"
- board text added: "PA31"
- board text added: "PB02"
- board text added: "PB03"
- board text added: "PB08"
- board text added: "PB09"
- board text added: "PB10"
- board text added: "PB11"
- board text added: "PB22"
- board text added: "PB23"
- board text removed: "A/C"
- board text removed: "A0"
- board text removed: "A2"
- board text removed: "A3"
- board text removed: "A4"
- board text removed: "A5"
- board text removed: "AREF"
- board text removed: "SCL"
- board text removed: "SDA"
- board text removed: "SWCLK"
- board text removed: "SWDIO"

Commit message: final?
Parts:
- added J1: HV in, Connector_PinHeader_2.54mm:PinHeader_1x01_P2.54mm_Vertical, F.Cu at (207.3, 90.2)
- moved J21 52.3 mm to (195.3, 128.2), turned to -90 degrees
- moved J22 39.7 mm to (202.4, 128.2), turned to -90 degrees
- moved J8 29.7 mm to (158.6, 91.2), turned to 180 degrees
- moved BAR1 23.6 mm to (171.5, 68.3), turned to 0 degrees
- moved R14 23.3 mm to (167.4, 68.3), turned to 0 degrees
- moved R23 23.1 mm to (167.4, 91.2), turned to 0 degrees
- moved R15 18.3 mm to (167.4, 70.9), turned to 0 degrees
- moved R22 18.2 mm to (167.4, 88.7), turned to 0 degrees
- moved R16 13.4 mm to (167.4, 73.4), turned to 0 degrees
- moved R21 13.3 mm to (167.4, 86.1), turned to 0 degrees
- moved R17 8.67 mm to (167.4, 76.0), turned to 0 degrees
- moved R20 8.55 mm to (167.4, 83.6), turned to 0 degrees
- moved R18 4.78 mm to (167.4, 78.5), turned to 0 degrees
- moved R19 4.71 mm to (167.4, 81.0), turned to 0 degrees
- moved JP1 1.41 mm to (155.9, 123.3)
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Connections:
- J45 pad 1: Net-(J45-Pin_1) -> Net-(J1-Pin_1)
- J45 pad 10: Net-(J45-Pin_10) -> Net-(J1-Pin_1)
- J45 pad 11: Net-(J45-Pin_11) -> Net-(J1-Pin_1)
- J45 pad 12: Net-(J45-Pin_11) -> Net-(J1-Pin_1)
- J45 pad 13: Net-(J45-Pin_13) -> Net-(J1-Pin_1)
- J45 pad 14: Net-(J45-Pin_13) -> Net-(J1-Pin_1)
- J45 pad 15: Net-(J45-Pin_15) -> Net-(J1-Pin_1)
- J45 pad 16: Net-(J45-Pin_15) -> Net-(J1-Pin_1)
- J45 pad 17: Net-(J45-Pin_17) -> Net-(J1-Pin_1)
- J45 pad 18: Net-(J45-Pin_17) -> Net-(J1-Pin_1)
- J45 pad 2: Net-(J45-Pin_1) -> Net-(J1-Pin_1)
- J45 pad 3: Net-(J45-Pin_3) -> Net-(J1-Pin_1)
- J45 pad 4: Net-(J45-Pin_3) -> Net-(J1-Pin_1)
- J45 pad 5: Net-(J45-Pin_5) -> Net-(J1-Pin_1)
- J45 pad 6: Net-(J45-Pin_5) -> Net-(J1-Pin_1)
- J45 pad 7: Net-(J45-Pin_7) -> Net-(J1-Pin_1)
- J45 pad 8: Net-(J45-Pin_7) -> Net-(J1-Pin_1)
- J45 pad 9: Net-(J45-Pin_10) -> Net-(J1-Pin_1)
Routing:
- net Net-(J1-Pin_1): track 0.00 -> 56.6 mm
- net GND: track 676.0 -> 650.5 mm
- net Net-(J45-Pin_7): track 2.54 -> 0.00 mm
- net Net-(J45-Pin_5): track 2.54 -> 0.00 mm
- net Net-(J45-Pin_3): track 2.54 -> 0.00 mm
- net Net-(J45-Pin_17): track 2.54 -> 0.00 mm
- net Net-(J45-Pin_15): track 2.54 -> 0.00 mm
- net Net-(J45-Pin_13): track 2.54 -> 0.00 mm
- net Net-(J45-Pin_11): track 2.54 -> 0.00 mm
- net Net-(J45-Pin_10): track 2.54 -> 0.00 mm
- net Net-(J45-Pin_1): track 2.54 -> 0.00 mm
- net Net-(J8-Pin_5): track 5.39 -> 7.82 mm
- net Net-(J8-Pin_7): track 5.39 -> 7.82 mm
- net Net-(J8-Pin_9): track 5.39 -> 7.82 mm
- net Net-(J8-Pin_8): track 5.39 -> 7.82 mm
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Other:
- board text added: "HV IN"
- board text added: "LCD Voltage"
- board text added: "LED1"
- board text added: "LED10"
- board text added: "LED2"
- board text added: "LED3"
- board text added: "LED4"
- board text added: "LED5"
- board text added: "LED6"
- board text added: "LED7"
- board text added: "LED8"
- board text added: "LED9"
- board text added: "RE-A"
- board text added: "RE-B"
- board text added: "RE-P"
- board text added: "SW1"
